Commit message: Asset Management and File Path Modification

File: ur5e_robotiq.urdf (robot description, URDF)
Before this commit: robot ur5e_robot, 22 links, 21 joints
Links:
- link base_link_inertia: geometry collision mesh filename=assets/ur5e/collision/base.stl; visual mesh filename=assets/ur5e/visual/base.dae
- link forearm_link: geometry collision mesh filename=assets/ur5e/collision/forearm.stl; visual mesh filename=assets/ur5e/visual/forearm.dae
- link left_inner_finger: geometry collision mesh filename=assets/robotiq_2f_85/meshes/collision/robotiq_arg2f_85_inne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 scale=0.001 0.001 0.001; visual mesh filename=assets/robotiq_2f_85/meshes/visual/robotiq_arg2f_85_inner_f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 scale=0.001 0.001 0.001
- link left_inner_knuckle: geometry collision mesh filename=assets/robotiq_2f_85/meshes/collision/robotiq_arg2f_85_inne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 scale=0.001 0.001 0.001; visual mesh filename=assets/robotiq_2f_85/meshes/visual/robotiq_arg2f_85_inner_k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 scale=0.001 0.001 0.001
- link left_outer_finger: geometry collision mesh filename=assets/robotiq_2f_85/meshes/collision/robotiq_arg2f_85_oute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 scale=0.001 0.001 0.001; visual mesh filename=assets/robotiq_2f_85/meshes/visual/robotiq_arg2f_85_outer_f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 scale=0.001 0.001 0.001
- link left_outer_knuckle: geometry collision mesh filename=assets/robotiq_2f_85/meshes/collision/robotiq_arg2f_85_oute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 scale=0.001 0.001 0.001; visual mesh filename=assets/robotiq_2f_85/meshes/visual/robotiq_arg2f_85_outer_k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 scale=0.001 0.001 0.001
- link right_inner_finger: geometry collision mesh filename=assets/robotiq_2f_85/meshes/collision/robotiq_arg2f_85_inne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 scale=0.001 0.001 0.001; visual mesh filename=assets/robotiq_2f_85/meshes/visual/robotiq_arg2f_85_inner_f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 scale=0.001 0.001 0.001
- link right_inner_knuckle: geometry collision mesh filename=assets/robotiq_2f_85/meshes/collision/robotiq_arg2f_85_inne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 scale=0.001 0.001 0.001; visual mesh filename=assets/robotiq_2f_85/meshes/visual/robotiq_arg2f_85_inner_k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 scale=0.001 0.001 0.001
- link right_outer_finger: geometry collision mesh filename=assets/robotiq_2f_85/meshes/collision/robotiq_arg2f_85_oute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 scale=0.001 0.001 0.001; visual mesh filename=assets/robotiq_2f_85/meshes/visual/robotiq_arg2f_85_outer_f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 scale=0.001 0.001 0.001
- link right_outer_knuckle: geometry collision mesh filename=assets/robotiq_2f_85/meshes/collision/robotiq_arg2f_85_oute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 scale=0.001 0.001 0.001; visual mesh filename=assets/robotiq_2f_85/meshes/visual/robotiq_arg2f_85_outer_k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 scale=0.001 0.001 0.001
- link robotiq_arg2f_base_link: geometry collision mesh filename=assets/robotiq_2f_85/meshes/collision/robotiq_arg2f_base_li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; visual mesh filename=assets/robotiq_2f_85/meshes/visual/robotiq_arg2f_85_base_li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 scale=0.001 0.001 0.001
- link shoulder_link: geometry collision mesh filename=assets/ur5e/collision/shoulder.stl; visual mesh filename=assets/ur5e/visual/shoulder.dae
- link upper_arm_link: geometry collision mesh filename=assets/ur5e/collision/upperarm.stl; visual mesh filename=assets/ur5e/visual/upperarm.dae
- link wrist_1_link: geometry collision mesh filename=assets/ur5e/collision/wrist1.stl; visual mesh filename=assets/ur5e/visual/wrist1.dae
- link wrist_2_link: geometry collision mesh filename=assets/ur5e/collision/wrist2.stl; visual mesh filename=assets/ur5e/visual/wrist2.dae
- link wrist_3_link: geometry collision mesh filename=assets/ur5e/collision/wrist3.stl; visual mesh filename=assets/ur5e/visual/wrist3.dae
